File: analog_switch_v1/analog_switch_v1.kicad_pcb (KiCad board)
At the start: 2 copper layers, 19 x 100 mm, 46 parts, among them J1 Conn_02x05_Odd_Even, J2 Audio In, J3 Audio Out, J4 Gate In, Q1 BC547, Q2 BC547, Q3 BC547, SW1 SW_GATE, U1 L78L05_SOT89, U2 TL072, U3 DG418LDJ

Commit message: Geographic re-annotate and silkscreen cleanup
Parts:
- moved LOGO101 80.8 mm to (149.4, 62.9)
- moved LOGO100 68.5 mm to (143.9, 78.3)
- moved LOGO102 54.7 mm to (142.8, 141.5), turned to 90 degrees
- moved R12 7.40 mm to (142.7, 125.7)
- moved R14 3.15 mm to (141.7, 131.3)
- renumbered C5 to C100, C4 to C101, C3 to C102, C6 to C103, C10 to C104, C9 to C105, C11 to C106, C8 to C107, C7 to C108, C1 to C3, D4 to D100, D3 to D2, D2 to D3, D1 to D4, FB2 to FB1, FB1 to FB2, J4 to J100, J2 to J101, J3 to J102, J1 to J2, LOGO3 to LOGO100, LOGO1 to LOGO101, LOGO2 to LOGO102, R9 to R1, R12 to R10, R15 to R12, R8 to R13, R2 to R14, R1 to R15, R10 to R2, R6 to R3, R7 to R4, R4 to R5, R5 to R6, R3 to R7, R14 to R8, R13 to R9, SW1 to SW100, U1 to U100, U3 to U2, U2 to U3
Routing:
- net Net-(D4-Pad1): track 91.6 -> 99.8 mm, vias 0 -> 1
- net Net-(Q3-Pad2): track 13.9 -> 8.36 mm
- net Net-(J101-PadT): track 11.9 -> 13.4 mm
- net Net-(D4-Pad2): track 5.32 -> 6.70 mm
Other:
- board text added: "Analog Switch"
- board text added: "Audio In"
- board text added: "Audio Out"
- board text added: "DG418LDJ"
- board text added: "Gate In"
- board text added: "L78L05"
- board text added: "Robot Dialogs"
- board text added: "TL072"
- board text added: "v1.0 Oct 2022"
- board text removed: "Eurorack Template"
- board text removed: "RobotDialogs"
- board text removed: "v1.1 July 2022"

Commit message: Tried to fix mystery fusion pcb issue
These boards had some issue when I ordered them, something in the
fusion pcb service didn't work right but I don't know what... So I
tweaked the silkscreen a bit and fixed the grid/drill origin. The
single pcb works in their system but it still complained about the
panelized version. I just submitted it anyways, we'll see if they find
some more specific issue.
Changed lines of the file:
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@@
     (pad_to_mask_clearance 0)
     (aux_axis_origin 140 150)
+    (grid_origin 140 150)
     (pcbplotparams
       (layerselection 0x00010fc_ffffffff)
@@
     )
     (fp_circle (center -4.4 0.1) (end -4.3 0.1) (layer "F.SilkS") (width 0.2) (fill none))
-    (fp_circle (center 0 0) (end 5 0) (layer "F.SilkS") (width 0.127) (fill none))
+    (fp_circle (center 0 0) (end 4.75 0) (layer "F.SilkS") (width 0.127) (fill none))
     (fp_circle (center 0 0) (end 5.25 0) (layer "F.CrtYd") (width 0.05) (fill none))
     (fp_circle (center 0 0) (end 5 0) (layer "F.Fab") (width 0.127) (fill none))
@@
     )
     (fp_line (start -0.9 -5.6) (end -4.5 -5.6) (layer "F.SilkS") (width 0.12))
-    (fp_line (start 4 4.5) (end 2.7 4.5) (layer "F.SilkS") (width 0.12))
+    (fp_line (start 3.4 4.5) (end 2.7 4.5) (layer "F.SilkS") (width 0.12))
     (fp_line (start -4.5 -5.6) (end -4.5 -1.35) (layer "F.SilkS") (width 0.12))
-    (fp_line (start 4 -5.6) (end 3 -5.6) (layer "F.SilkS") (width 0.12))
+    (fp_line (start 3.4 -5.6) (end 3 -5.6) (layer "F.SilkS") (width 0.12))
     (fp_line (start -4.5 4.5) (end -0.85 4.5) (layer "F.SilkS") (width 0.12))
-    (fp_line (start 4 4.5) (end 4 -5.6) (layer "F.SilkS") (width 0.12))
+    (fp_line (start 3.4 4.5) (end 3.4 -5.6) (layer "F.SilkS") (width 0.12))
     (fp_line (start -4.5 3.15) (end -4.5 4.5) (layer "F.SilkS") (width 0.12))
     (fp_arc (start -2.673091 -1.311329) (mid 1.644329 -2.482173) (end 2.25 1.95) (layer "F.SilkS") (width 0.12))
@@
     (style (thickness 0.1) (arrow_length 1.27) (text_position_mode 0) (extension_height 0.58642) (extension_offset 0.5) keep_text_aligned)
   )
-  (dimension locked (type aligned) (layer "F.Fab")
-    (pts (xy 159 123.8) (xy 159 109.8))
+  (dimension (type aligned) (layer "F.Fab")
+    (pts (xy 159 123.8) (xy 159 116.5))
     (height -22)
-    (gr_text "14.0000 mm" (at 135.85 116.8 90) (layer "F.Fab")
-      (effects (font (size 1 1) (thickness 0.15)))
-    )
+    (gr_text "7.3000 mm" (at 135.85 120.15 90) (layer "F.Fab")
+      (effects (font (size 1 1) (thickness 0.15)))
+    )
